File: PCBs/Lower Board/Euclid_Lower.sch (EAGLE design)
At the start: 28 parts, among them J1 USB_B, J3 USB_A_PTH_MALE

Commit message: New version with sample file support
Parts:
- D15: value (none) -> 1n4148
Changed lines of the file:
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@@
 <?xml version="1.0" encoding="utf-8"?>
 <!DOCTYPE eagle SYSTEM "eagle.dtd">
-<eagle version="6.1">
+<eagle version="8.2.1">
 <drawing>
 <settings>
@@
 <part name="J4" library="SparkFun-Connectors" deviceset="CONN_02" device=""/>
 <part name="LINE_OUT" library="SparkFun-Connectors" deviceset="AUDIO_JACK_3.5MM" device="_KIT" value=""/>
-<part name="D15" library="adafruit" deviceset="DIODE" device="DO-1N4148"/>
+<part name="D15" library="adafruit" deviceset="DIODE" device="DO-1N4148" value="1n4148"/>
 <part name="SV1" library="con-lstb" deviceset="MA10-2" device=""/>
 <part name="SUPPLY2" library="supply2" deviceset="VCC" device=""/>
