File: PCBs/Upper Board/Euclid_Upper.brd (EAGLE design)
At the start: 181.6 x 132.1 mm, 85 parts, among them IC1 MCP23017SO, IC2 MCP23017SO, IC3 MCP23017SO, IC4 MCP23017SO

Commit message: New version with sample file support
Parts:
- removed BRIGHTNESS: 1K, pot:CT6
Connections:
- removed net N$2: BRIGHTNESS.S, R10.2, R11.2, R12.2, R13.2, R14.2, R15.2, R16.2, R17.2, R18.2, R19.2, R2.2, R20.2, R21.2, R22.2, R23.2, R24.2, R25.2, R26.2, R27.2, R28.2, R29.2, R3.2, R30.2, R4.2, R6.2, R7.2, R8.2, R9.2
- net GND: now also R10.2, R11.2, R12.2, R13.2, R14.2, R15.2, R16.2, R17.2, R18.2, R19.2, R2.2, R20.2, R21.2, R22.2, R23.2, R24.2, R25.2, R26.2, R27.2, R28.2, R29.2, R3.2, R30.2, R4.2, R6.2, R7.2, R8.2, R9.2; no longer BRIGHTNESS.A
- net VCC: no longer BRIGHTNESS.E
Routing:
- net N$2: track 646.3 -> 0.00 mm
- net GND: track 942.5 -> 1518.3 mm
- net VCC: track 568.6 -> 551.1 mm
