File: PCBs/Upper Board/Euclid_Upper.sch (EAGLE design)
At the start: 85 parts, among them IC1 MCP23017SO, IC2 MCP23017SO, IC3 MCP23017SO, IC4 MCP23017SO

Commit message: New version with sample file support
Parts:
- removed BRIGHTNESS: 1K, pot:TRIM_EU-CT6
Connections:
- removed net N$2: BRIGHTNESS.S, R10.2, R11.2, R12.2, R13.2, R14.2, R15.2, R16.2, R17.2, R18.2, R19.2, R2.2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
- net GND: now also R10.2, R11.2, R12.2, R13.2, R14.2, R15.2, R16.2, R17.2, R18.2, R19.2, R2.2, R20.2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; no longer BRIGHTNESS.A
- net VCC: no longer BRIGHTNESS.E
